File: hardware/audio_iface/vu_meter.kicad_sch (KiCad schematic)
At the start: 34 parts, among them U501 MCP23S17-E/SO

Commit message: crude placement
Connections:
- net GPB0: now reaches D501.1 (K), U501.1 (GPB0)
- net GPA7: now reaches D516.1 (K), U501.28 (GPA7)
- net GPA5: now reaches D514.1 (K), U501.26 (GPA5)
- net GPA0: now reaches D509.1 (K), U501.21 (GPA0)
- net GPA6: now reaches D515.1 (K), U501.27 (GPA6)
- net GPB5: now reaches D506.1 (K), U501.6 (GPB5)
- net GPB3: now reaches D504.1 (K), U501.4 (GPB3)
- net GPB1: now reaches D502.1 (K), U501.2 (GPB1)
- net GPA1: now reaches D510.1 (K), U501.22 (GPA1)
- net GPB2: now reaches D503.1 (K), U501.3 (GPB2)
- net GPA4: now reaches D513.1 (K), U501.25 (GPA4)
- net GPB6: now reaches D507.1 (K), U501.7 (GPB6)
- net GPA2: now reaches D511.1 (K), U501.23 (GPA2)
- net GPB7: now reaches D508.1 (K), U501.8 (GPB7)
- net GPA3: now reaches D512.1 (K), U501.24 (GPA3)
- net GPB4: now reaches D505.1 (K), U501.5 (GPB4)
Changed lines of the file:
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@@
+    (effects (font (size 1.27 1.27)) (justify left bottom))
+  )
+  (label "GPA1" (at 148.59 104.14 0) (fields_autoplaced)
+    (effects (font (size 1.27 1.27)) (justify left bottom))
+  )
+  (label "GPB4" (at 148.59 88.9 0) (fields_autoplaced)
+    (effects (font (size 1.27 1.27)) (justify left bottom))
+  )
+  (label "GPA3" (at 148.59 109.22 0) (fields_autoplaced)
+    (effects (font (size 1.27 1.27)) (justify left bottom))
+  )
+  (label "GPA5" (at 152.4 120.65 0) (fields_autoplaced)
+    (effects (font (size 1.27 1.27)) (justify left bottom))
+  )
+  (label "GPB1" (at 153.67 73.66 0) (fields_autoplaced)
+    (effects (font (size 1.27 1.27)) (justify left bottom))
+  )
+  (label "GPA0" (at 148.59 101.6 0) (fields_autoplaced)
+    (effects (font (size 1.27 1.27)) (justify left bottom))
+  )
+  (label "GPA4" (at 148.59 111.76 0) (fields_autoplaced)
+    (effects (font (size 1.27 1.27)) (justify left bottom))
+  )
+  (label "GPB6" (at 148.59 93.98 0) (fields_autoplaced)
+    (effects (font (size 1.27 1.27)) (justify left bottom))
+  )
+  (label "GPA7" (at 152.3679 128.27 0) (fields_autoplaced)
+    (effects (font (size 1.27 1.27)) (justify left bottom))
+  )
+  (label "GPB0" (at 153.67 69.85 0) (fields_autoplaced)
+    (effects (font (size 1.27 1.27)) (justify left bottom))
+  )
+  (label "GPB5" (at 148.59 91.44 0) (fields_autoplaced)
+    (effects (font (size 1.27 1.27)) (justify left bottom))
+  )
+  (label "GPB3" (at 153.67 81.28 0) (fields_autoplaced)
+    (effects (font (size 1.27 1.27)) (justify left bottom))
+  )
+  (label "GPB2" (at 153.67 77.47 0) (fields_autoplaced)
+    (effects (font (size 1.27 1.27)) (justify left bottom))
+  )
+  (label "GPA2" (at 148.59 106.68 0) (fields_autoplaced)
+    (effects (font (size 1.27 1.27)) (justify left bottom))
+  )
+  (label "GPB7" (at 148.59 96.52 0) (fields_autoplaced)
+    (effects (font (size 1.27 1.27)) (justify left bottom))
+  )
+  (label "GPA6" (at 152.4 124.46 0) (fields_autoplaced)
     (effects (font (size 1.27 1.27)) (justify left bottom))
   )
