File: hardware/audio_iface/nucleo.kicad_sch (KiCad schematic)
At the start: 1 part, among them U101 NUCLEO_L476RG

Commit message: schematic v1 done
Parts:
- added J201: UART, Connector_JST:JST_XH_S3B-XH-A_1x03_P2.50mm_Horizontal, symbol Connector_Generic:Conn_01x03
- added TP301 (x4): TestPoint, Connector_Pin:Pin_D1.1mm_L8.5mm_W2.5mm_FlatFork, symbol Connector:TestPoint
Connections:
- net +3.3V: now also TP301.1
- net +3.3VA: now also TP301.1
- net GND: now also J201.3 (Pin_3)
- new net UART_RX: J201.1 (Pin_1), TP301.1
- new net UART_TX: J201.2 (Pin_2), TP301.1
Other:
- note added: "Wuerth 61304021821 Header femelle 40 pin"
Changed lines of the file:
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@@
   (junction (at 120.65 111.76) (diameter 0) (color 0 0 0 0)
   )
+  (junction (at 85.09 104.14) (diameter 0) (color 0 0 0 0)
+  )
   (junction (at 120.65 106.68) (diameter 0) (color 0 0 0 0)
   )
@@
   )
   (junction (at 120.65 119.38) (diameter 0) (color 0 0 0 0)
+  )
+  (junction (at 71.12 106.68) (diameter 0) (color 0 0 0 0)
   )
   (junction (at 120.65 109.22) (diameter 0) (color 0 0 0 0)
@@
   (no_connect (at 92.71 96.52))
   (no_connect (at 92.71 116.84))
-  (wire (pts (xy 92.71 106.68) (xy 77.47 106.68))
+  (wire (pts (xy 92.71 106.68) (xy 71.12 106.68))
+    (stroke (width 0) (type default))
+  )
+  (wire (pts (xy 85.09 34.29) (xy 93.98 34.29))
     (stroke (width 0) (type default))
   )
@@
     (stroke (width 0) (type default))
   )
+  (wire (pts (xy 86.36 40.64) (xy 86.36 39.37))
+    (stroke (width 0) (type default))
+  )
   (wire (pts (xy 85.09 104.14) (xy 92.71 104.14))
     (stroke (width 0) (type default))
   )
+  (wire (pts (xy 85.09 36.83) (xy 93.98 36.83))
+    (stroke (width 0) (type default))
+  )
   (wire (pts (xy 120.65 109.22) (xy 120.65 106.68))
     (stroke (width 0) (type default))
   )
+  (wire (pts (xy 86.36 39.37) (xy 85.09 39.37))
+    (stroke (width 0) (type default))
+  )
   (wire (pts (xy 118.11 119.38) (xy 120.65 119.38))
     (stroke (width 0) (type default))
   )
-  (wire (pts (xy 77.47 106.68) (xy 77.47 102.87))
+  (wire (pts (xy 71.12 106.68) (xy 71.12 102.87))
     (stroke (width 0) (type default))
   )
@@
   (wire (pts (xy 118.11 116.84) (xy 120.65 116.84))
     (stroke (width 0) (type default))
+  )
+  (text "Wuerth 61304021821\nHeader femelle 40 pin" (at 109.22 76.2 0)
+    (effects (font (size 1.27 1.27)) (justify left bottom))
   )
   (text "On veut pouvoir l'alimenter depuis l'USB de la nucleo\n(Pour faire des TP sans brancher l'USB-C de l'audio)"
@@
     (effects (font (size 1.27 1.27)) (justify left bottom))
   )
+  (label "UART_TX" (at 224.79 93.98 0) (fields_autoplaced)
+    (effects (font (size 1.27 1.27)) (justify left bottom))
+  )
+  (label "UART_RX" (at 85.09 34.29 0) (fields_autoplaced)
+    (effects (font (size 1.27 1.27)) (justify left bottom))
+  )
+  (label "UART_RX" (at 224.79 91.44 0) (fields_autoplaced)
+    (effects (font (size 1.27 1.27)) (justify left bottom))
+  )
+  (label "UART_TX" (at 85.09 36.83 0) (fields_autoplaced)
+    (effects (font (size 1.27 1.27)) (justify left bottom))
+  )
   (hierarchical_label "I2S_SCLK" (shape input) (at 240.03 50.8 180) (fields_autoplaced)
     (effects (font (size 1.27 1.27)) (justify right))
@@
     (effects (font (size 1.27 1.27)) (justify right))
   )
+  (symbol (lib_id "power:GND") (at 86.36 40.64 0) (unit 1)
+    (in_bom yes) (on_board yes) (dnp no) (fields_autoplaced)
+    (property "Reference" "#PWR0204" (at 86.36 46.99 0)
+      (effects (font (size 1.27 1.27)) hide)
+    )
+    (property "Value" "GND" (at 86.36 45.72 0)
+      (effects (font (size 1.27 1.27)))
+    )
+    (property "Footprint" "" (at 86.36 40.64 0)
+      (effects (font (size 1.27 1.27)) hide)
+    )
+    (property "Datasheet" "" (at 86.36 40.64 0)
+      (effects (font (size 1.27 1.27)) hide)
+    )
+    (pin "1")
+    (instances
+      (project "audio_iface"
+        (path "/84adbf2e-65c7-4710-86f9-725cae0256c9/cdd727d1-dc6e-479c-822a-c88c05fafe87"
+          (reference "#PWR0204") (unit 1)
+        )
+      )
+    )
+  )
   (symbol (lib_id "power:+3.3VA") (at 85.09 102.87 0) (unit 1)
     (in_bom yes) (on_board yes) (dnp no) (fields_autoplaced)
@@
         (path "/84adbf2e-65c7-4710-86f9-725cae0256c9/cdd727d1-dc6e-479c-822a-c88c05fafe87"
           (reference "#PWR0202") (unit 1)
+        )
+      )
+    )
+  )
+  (symbol (lib_id "Connector:TestPoint") (at 85.09 104.14 90) (unit 1)
+    (in_bom yes) (on_board yes) (dnp no)
+    (property "Reference" "TP301" (at 80.01 104.14 90)
+      (effects (font (size 1.27 1.27)) (justify left))
+    )
+    (property "Value" "TestPoint" (at 83.058 101.6 0)
+      (effects (font (size 1.27 1.27)) (justify left) hide)
+    )
+    (property "Footprint" "Connector_Pin:Pin_D1.1mm_L8.5mm_W2.5mm_FlatFork" (at 85.09 99.06 0)
+      (effects (font (size 1.27 1.27)) hide)
+    )
+    (property "Datasheet" "~" (at 85.09 99.06 0)
+      (effects (font (size 1.27 1.27)) hide)
+    )
+    (pin "1")
+    (instances
+      (project "audio_iface"
+        (path "/84adbf2e-65c7-4710-86f9-725cae0256c9/b36b6a55-ed48-4879-90b2-e55dd522c7e4"
+          (reference "TP301") (unit 1)
+        )
+        (path "/84adbf2e-65c7-4710-86f9-725cae0256c9"
+          (reference "TP108") (unit 1)
+        )
+        (path "/84adbf2e-65c7-4710-86f9-725cae0256c9/cdd727d1-dc6e-479c-822a-c88c05fafe87"
+          (reference "TP202") (unit 1)
+        )
+      )
+    )
+  )
+  (symbol (lib_id "Connector:TestPoint") (at 93.98 34.29 270) (unit 1)
+    (in_bom yes) (on_board yes) (dnp no)
+    (property "Reference" "TP301" (at 99.06 34.29 90)
+      (effects (font (size 1.27 1.27)) (justify left))
+    )
+    (property "Value" "TestPoint" (at 96.012 36.83 0)
+      (effects (font (size 1.27 1.27)) (justify left) hide)
+    )
+    (property "Footprint" "Connector_Pin:Pin_D1.1mm_L8.5mm_W2.5mm_FlatFork" (at 93.98 39.37 0)
+      (effects (font (size 1.27 1.27)) hide)
+    )
+    (property "Datasheet" "~" (at 93.98 39.37 0)
+      (effects (font (size 1.27 1.27)) hide)
+    )
+    (pin "1")
+    (instances
+      (project "audio_iface"
+        (path "/84adbf2e-65c7-4710-86f9-725cae0256c9/b36b6a55-ed48-4879-90b2-e55dd522c7e4"
+          (reference "TP301") (unit 1)
+        )
+        (path "/84adbf2e-65c7-4710-86f9-725cae0256c9"
+          (reference "TP108") (unit 1)
+        )
+        (path "/84adbf2e-65c7-4710-86f9-725cae0256c9/cdd727d1-dc6e-479c-822a-c88c05fafe87"
+          (reference "TP203") (unit 1)
+        )
+      )
+    )
+  )
+  (symbol (lib_id "Connector:TestPoint") (at 71.12 106.68 90) (unit 1)
+    (in_bom yes) (on_board yes) (dnp no)
+    (property "Reference" "TP301" (at 66.04 106.68 90)
+      (effects (font (size 1.27 1.27)) (justify left))
+    )
+    (property "Value" "TestPoint" (at 69.088 104.14 0)
+      (effects (font (size 1.27 1.27)) (justify left) hide)
+    )
+    (property "Footprint" "Connector_Pin:Pin_D1.1mm_L8.5mm_W2.5mm_FlatFork" (at 71.12 101.6 0)
+      (effects (font (size 1.27 1.27)) hide)
+    )
+    (property "Datasheet" "~" (at 71.12 101.6 0)
+      (effects (font (size 1.27 1.27)) hide)
+    )
+    (pin "1")
+    (instances
+      (project "audio_iface"
+        (path "/84adbf2e-65c7-4710-86f9-725cae0256c9/b36b6a55-ed48-4879-90b2-e55dd522c7e4"
+          (reference "TP301") (unit 1)
+        )
+        (path "/84adbf2e-65c7-4710-86f9-725cae0256c9"
+          (reference "TP108") (unit 1)
+        )
+        (path "/84adbf2e-65c7-4710-86f9-725cae0256c9/cdd727d1-dc6e-479c-822a-c88c05fafe87"
+          (reference "TP201") (unit 1)
+        )
+      )
+    )
+  )
+  (symbol (lib_id "Connector_Generic:Conn_01x03") (at 80.01 36.83 0) (mirror y) (unit 1)
+    (in_bom yes) (on_board yes) (dnp no) (fields_autoplaced)
+    (property "Reference" "J201" (at 80.01 27.94 0)
+      (effects (font (size 1.27 1.27)))
+    )
+    (property "Value" "UART" (at 80.01 30.48 0)
+      (effects (font (size 1.27 1.27)))
+    )
+    (property "Footprint" "Connector_JST:JST_XH_S3B-XH-A_1x03_P2.50mm_Horizontal" (at 80.01 36.83 0)
+      (effects (font (size 1.27 1.27)) hide)
+    )
+    (property "Datasheet" "~" (at 80.01 36.83 0)
+      (effects (font (size 1.27 1.27)) hide)
+    )
+    (pin "1")
+    (pin "2")
+    (pin "3")
+    (instances
+      (project "audio_iface"
+        (path "/84adbf2e-65c7-4710-86f9-725cae0256c9/cdd727d1-dc6e-479c-822a-c88c05fafe87"
+          (reference "J201") (unit 1)
         )
       )
@@
     )
   )
-  (symbol (lib_id "power:+3.3V") (at 77.47 102.87 0) (unit 1)
-    (in_bom yes) (on_board yes) (dnp no) (fields_autoplaced)
-    (property "Reference" "#PWR0201" (at 77.47 106.68 0)
-      (effects (font (size 1.27 1.27)) hide)
-    )
-    (property "Value" "+3.3V" (at 77.47 99.06 0)
-      (effects (font (size 1.27 1.27)))
-    )
-    (property "Footprint" "" (at 77.47 102.87 0)
-      (effects (font (size 1.27 1.27)) hide)
-    )
-    (property "Datasheet" "" (at 77.47 102.87 0)
-      (effects (font (size 1.27 1.27)) hide)
-    )
+  (symbol (lib_id "Connector:TestPoint") (at 93.98 36.83 270) (unit 1)
+    (in_bom yes) (on_board yes) (dnp no)
+    (property "Reference" "TP301" (at 99.06 36.83 90)
+      (effects (font (size 1.27 1.27)) (justify left))
+    )
+    (property "Value" "TestPoint" (at 96.012 39.37 0)
+      (effects (font (size 1.27 1.27)) (justify left) hide)
+    )
+    (property "Footprint" "Connector_Pin:Pin_D1.1mm_L8.5mm_W2.5mm_FlatFork" (at 93.98 41.91 0)
+      (effects (font (size 1.27 1.27)) hide)
+    )
+    (property "Datasheet" "~" (at 93.98 41.91 0)
+      (effects (font (size 1.27 1.27)) hide)
+    )
+    (pin "1")
+    (instances
+      (project "audio_iface"
+        (path "/84adbf2e-65c7-4710-86f9-725cae0256c9/b36b6a55-ed48-4879-90b2-e55dd522c7e4"
+          (reference "TP301") (unit 1)
+        )
+        (path "/84adbf2e-65c7-4710-86f9-725cae0256c9"
+          (reference "TP108") (unit 1)
+        )
+        (path "/84adbf2e-65c7-4710-86f9-725cae0256c9/cdd727d1-dc6e-479c-822a-c88c05fafe87"
+          (reference "TP204") (unit 1)
+        )
+      )
+    )
+  )
+  (symbol (lib_id "power:+3.3V") (at 71.12 102.87 0) (unit 1)
+    (in_bom yes) (on_board yes) (dnp no) (fields_autoplaced)
+    (property "Reference" "#PWR0201" (at 71.12 106.68 0)
+      (effects (font (size 1.27 1.27)) hide)
+    )
+    (property "Value" "+3.3V" (at 71.12 99.06 0)
+      (effects (font (size 1.27 1.27)))
+    )
+    (property "Footprint" "" (at 71.12 102.87 0)
+      (effects (font (size 1.27 1.27)) hide)
+    )
+    (property "Datasheet" "" (at 71.12 102.87 0)
+      (effects (font (size 1.27 1.27)) hide)
+    )

Commit message: crude placement
Parts:
- TP301: value TestPoint -> +3.3VA
- TP301: value TestPoint -> RX
- TP301: value TestPoint -> +3.3V
- TP301: value TestPoint -> TX
Connections:
- net I2C_SCL: now also U101.225 (PB10)
- net I2C_SDA: now also U101.218 (PB11)
- net I2S_DIN: now also U101.226 (PB15)
- net I2S_DOUT: now also U101.103 (PC12)
- net I2S_LRCLK: now also U101.216 (PB12)
- net I2S_SCLK: now also U101.230 (PB13)
- net SYS_MCLK: now also U101.228 (PB14)
- net UART_RX: now also U101.233 (PA10)
- net UART_TX: now also U101.221 (PA9)
- net VU_MISO: now also U101.102 (PC11)
- net VU_MOSI: now also U101.229 (PB5)
- net VU_SCK: now also U101.101 (PC10)
- net VU_nCS: now also U101.217 (PB6)
- net VU_nRESET: now also U101.121 (PB7)
Changed lines of the file:
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@@
     (effects (font (size 1.27 1.27)) (justify left bottom))
   )
-  (label "UART_TX" (at 224.79 93.98 0) (fields_autoplaced)
-    (effects (font (size 1.27 1.27)) (justify left bottom))
+  (label "UART_TX" (at 152.4 90.17 180) (fields_autoplaced)
+    (effects (font (size 1.27 1.27)) (justify right bottom))
   )
   (label "UART_RX" (at 85.09 34.29 0) (fields_autoplaced)
     (effects (font (size 1.27 1.27)) (justify left bottom))
   )
-  (label "UART_RX" (at 224.79 91.44 0) (fields_autoplaced)
-    (effects (font (size 1.27 1.27)) (justify left bottom))
+  (label "UART_RX" (at 152.4 92.71 180) (fields_autoplaced)
+    (effects (font (size 1.27 1.27)) (justify right bottom))
   )
   (label "UART_TX" (at 85.09 36.83 0) (fields_autoplaced)
     (effects (font (size 1.27 1.27)) (justify left bottom))
   )
-  (hierarchical_label "I2S_SCLK" (shape input) (at 240.03 50.8 180) (fields_autoplaced)
-    (effects (font (size 1.27 1.27)) (justify right))
-  )
-  (hierarchical_label "VU_MOSI" (shape input) (at 232.41 121.92 180) (fields_autoplaced)
-    (effects (font (size 1.27 1.27)) (justify right))
-  )
-  (hierarchical_label "I2S_DIN" (shape input) (at 240.03 55.88 180) (fields_autoplaced)
-    (effects (font (size 1.27 1.27)) (justify right))
-  )
-  (hierarchical_label "I2S_DOUT" (shape input) (at 240.03 53.34 180) (fields_autoplaced)
-    (effects (font (size 1.27 1.27)) (justify right))
-  )
-  (hierarchical_label "VU_nCS" (shape input) (at 232.41 116.84 180) (fields_autoplaced)
-    (effects (font (size 1.27 1.27)) (justify right))
-  )
-  (hierarchical_label "I2C_SCL" (shape input) (at 241.3 62.23 180) (fields_autoplaced)
-    (effects (font (size 1.27 1.27)) (justify right))
-  )
-  (hierarchical_label "I2C_SDA" (shape input) (at 241.3 59.69 180) (fields_autoplaced)
-    (effects (font (size 1.27 1.27)) (justify right))
-  )
-  (hierarchical_label "VU_MISO" (shape input) (at 232.41 124.46 180) (fields_autoplaced)
-    (effects (font (size 1.27 1.27)) (justify right))
-  )
-  (hierarchical_label "VU_nRESET" (shape input) (at 232.41 139.7 180) (fields_autoplaced)
+  (hierarchical_label "I2S_SCLK" (shape input) (at 152.4 143.51 180) (fields_autoplaced)
+    (effects (font (size 1.27 1.27)) (justify right))
+  )
+  (hierarchical_label "VU_MOSI" (shape input) (at 152.4 123.19 180) (fields_autoplaced)
+    (effects (font (size 1.27 1.27)) (justify right))
+  )
+  (hierarchical_label "I2S_DIN" (shape input) (at 152.4 148.59 180) (fields_autoplaced)
+    (effects (font (size 1.27 1.27)) (justify right))
+  )
+  (hierarchical_label "I2S_DOUT" (shape input) (at 180.34 97.79 0) (fields_autoplaced)
+    (effects (font (size 1.27 1.27)) (justify left))
+  )
+  (hierarchical_label "VU_nCS" (shape input) (at 152.4 125.73 180) (fields_autoplaced)
+    (effects (font (size 1.27 1.27)) (justify right))
+  )
+  (hierarchical_label "I2C_SCL" (shape input) (at 152.4 135.89 180) (fields_autoplaced)
+    (effects (font (size 1.27 1.27)) (justify right))
+  )
+  (hierarchical_label "I2C_SDA" (shape input) (at 152.4 138.43 180) (fields_autoplaced)
+    (effects (font (size 1.27 1.27)) (justify right))
+  )
+  (hierarchical_label "VU_MISO" (shape input) (at 180.34 95.25 0) (fields_autoplaced)
+    (effects (font (size 1.27 1.27)) (justify left))
+  )
+  (hierarchical_label "VU_nRESET" (shape input) (at 152.4 128.27 180) (fields_autoplaced)
     (effects (font (size 1.27 1.27)) (justify right))
   )
@@
     (effects (font (size 1.27 1.27)) (justify right))
   )
-  (hierarchical_label "SYS_MCLK" (shape input) (at 240.03 43.18 180) (fields_autoplaced)
+  (hierarchical_label "SYS_MCLK" (shape input) (at 152.4 146.05 180) (fields_autoplaced)
     (effects (font (size 1.27 1.27)) (justify right))
   )
@@
     (effects (font (size 1.27 1.27)) (justify right))
   )
-  (hierarchical_label "VU_SCK" (shape input) (at 232.41 119.38 180) (fields_autoplaced)
-    (effects (font (size 1.27 1.27)) (justify right))
-  )
-  (hierarchical_label "I2S_LRCLK" (shape input) (at 240.03 48.26 180) (fields_autoplaced)
+  (hierarchical_label "VU_SCK" (shape input) (at 180.34 92.71 0) (fields_autoplaced)
+    (effects (font (size 1.27 1.27)) (justify left))
+  )
+  (hierarchical_label "I2S_LRCLK" (shape input) (at 152.4 140.97 180) (fields_autoplaced)
     (effects (font (size 1.27 1.27)) (justify right))
   )
@@
       (effects (font (size 1.27 1.27)) (justify left))
     )
-    (property "Value" "TestPoint" (at 83.058 101.6 0)
+    (property "Value" "+3.3VA" (at 83.058 101.6 0)
       (effects (font (size 1.27 1.27)) (justify left) hide)
     )
@@
       (effects (font (size 1.27 1.27)) (justify left))
     )
-    (property "Value" "TestPoint" (at 96.012 36.83 0)
+    (property "Value" "RX" (at 96.012 36.83 0)
       (effects (font (size 1.27 1.27)) (justify left) hide)
     )
@@
       (effects (font (size 1.27 1.27)) (justify left))
     )
-    (property "Value" "TestPoint" (at 69.088 104.14 0)
+    (property "Value" "+3.3V" (at 69.088 104.14 0)
       (effects (font (size 1.27 1.27)) (justify left) hide)
     )
@@
       (effects (font (size 1.27 1.27)) (justify left))
     )
-    (property "Value" "TestPoint" (at 96.012 39.37 0)
+    (property "Value" "TX" (at 96.012 39.37 0)
       (effects (font (size 1.27 1.27)) (justify left) hide)
     )

Commit message: routing v1
Parts:
- added TP301: GND, Connector_Pin:Pin_D1.1mm_L8.5mm_W2.5mm_FlatFork, symbol Connector:TestPoint
Connections:
- net GND: now also TP301.1
- net VU_nCS: now also U101.121 (PB7); no longer U101.217 (PB6)
- net VU_nRESET: now also U101.128 (PA0); no longer U101.121 (PB7)
Changed lines of the file:
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@@
   (junction (at 120.65 109.22) (diameter 0) (color 0 0 0 0)
+  )
+  (junction (at 120.65 101.6) (diameter 0) (color 0 0 0 0)
   )
   (junction (at 120.65 114.3) (diameter 0) (color 0 0 0 0)
@@
     (stroke (width 0) (type default))
   )
+  (wire (pts (xy 120.65 100.33) (xy 120.65 101.6))
+    (stroke (width 0) (type default))
+  )
   (wire (pts (xy 120.65 111.76) (xy 120.65 109.22))
     (stroke (width 0) (type default))
@@
     (effects (font (size 1.27 1.27)) (justify left))
   )
-  (hierarchical_label "VU_nCS" (shape input) (at 152.4 125.73 180) (fields_autoplaced)
+  (hierarchical_label "VU_nCS" (shape input) (at 152.4 128.27 180) (fields_autoplaced)
     (effects (font (size 1.27 1.27)) (justify right))
   )
@@
     (effects (font (size 1.27 1.27)) (justify left))
   )
-  (hierarchical_label "VU_nRESET" (shape input) (at 152.4 128.27 180) (fields_autoplaced)
+  (hierarchical_label "VU_nRESET" (shape input) (at 152.4 67.31 180) (fields_autoplaced)
     (effects (font (size 1.27 1.27)) (justify right))
   )
@@
         )
       )
+    )
+  )
+  (symbol (lib_id "Connector:TestPoint") (at 120.65 100.33 0) (unit 1)
+    (in_bom yes) (on_board yes) (dnp no)
+    (property "Reference" "TP301" (at 120.65 95.25 90)
+      (effects (font (size 1.27 1.27)) (justify left))
+    )
+    (property "Value" "GND" (at 123.19 98.298 0)
+      (effects (font (size 1.27 1.27)) (justify left) hide)
+    )
+    (property "Footprint" "Connector_Pin:Pin_D1.1mm_L8.5mm_W2.5mm_FlatFork" (at 125.73 100.33 0)
+      (effects (font (size 1.27 1.27)) hide)
+    )
+    (property "Datasheet" "~" (at 125.73 100.33 0)
+      (effects (font (size 1.27 1.27)) hide)
+    )
+    (pin "1")
+    (instances
+      (project "audio_iface"
+        (path "/84adbf2e-65c7-4710-86f9-725cae0256c9/b36b6a55-ed48-4879-90b2-e55dd522c7e4"
+          (reference "TP301") (unit 1)
+        )
+        (path "/84adbf2e-65c7-4710-86f9-725cae0256c9"
+          (reference "TP108") (unit 1)
+        )
+        (path "/84adbf2e-65c7-4710-86f9-725cae0256c9/cdd727d1-dc6e-479c-822a-c88c05fafe87"
+          (reference "TP205") (unit 1)
+        )
+      )
